Commit message: Add files via upload

File: my_rover_description/urdf/my_rover.xacro (robot description, xacro)
@@ -2,5 +2,5 @@
 <robot name="my_rover" xmlns:xacro="http://www.ros.org/wiki/xacro">
   <xacro:include filename="$(find my_rover_description)/urdf/materials.xacro" />
-  <xacro:include filename="$(find my_rover_description)/urdf/my_rover.gazebo" />
+  <!-- <xacro:include filename="$(find my_rover_description)/urdf/my_rover.gazebo" /> -->
   <xacro:include filename="$(find my_rover_description)/urdf/macros.xacro" />
   <link name="link_chassis">
@@ -38,5 +38,5 @@
     </visual>
   </link>
-  <link name="sensor_laser">
+  <link name="laser">
     <inertial>
       <origin xyz="0 0 0" rpy="0 0 0" />
@@ -58,8 +58,8 @@
     </collision>
   </link>
-  <joint name="joint_sensor_laser" type="fixed">
+  <joint name="laser_joint" type="fixed">
     <origin xyz="0 0 0.125" rpy="0 0 0"/>
     <parent link="link_chassis"/>
-    <child link="sensor_laser"/>
+    <child link="laser"/>
   </joint>
   <xacro:link_wheel name="link_right_front_wheel" />
